File: PCB/PCB_HaSBot/robot2.kicad_sch (KiCad schematic)
At the start: 17 parts, among them J1 Conn_01x04, J2 Conn_01x04, J3 Conn_01x04, J4 Conn_01x04, J5 Conn_01x04, J6 Conn_01x04, J7 Conn_01x04, J8 Screw_Terminal_01x02, M1 Motor_Servo, U1 STM32F401RETx, U3 L7805

Commit message: Version 2.0 du PCB
Parts:
- removed U1: STM32F401RETx, Package_QFP:LQFP-64_10x10mm_P0.5mm, symbol MCU_ST_STM32F4:STM32F401RETx
- added H2: MountingHole_Pad, MountingHole:MountingHole_3.2mm_M3_DIN965_Pad, symbol Mechanical:MountingHole_Pad
- added J10, J11: Conn_01x08, Connector_PinHeader_2.54mm:PinHeader_1x08_P2.54mm_Vertical, symbol Connector_Generic:Conn_01x08
- added J12: Conn_01x06, Connector_PinHeader_2.54mm:PinHeader_1x06_P2.54mm_Vertical, symbol Connector_Generic:Conn_01x06
- added J9: Conn_01x10, Connector_PinHeader_2.54mm:PinHeader_1x10_P2.54mm_Vertical, symbol Connector_Generic:Conn_01x10
Connections:
- net +5V: now also J11.4 (Pin_4)
- net DIR_M1: now also J9.8 (Pin_8)
- net DIR_M2: now also J10.3 (Pin_3)
- net ENABLE_M1: now also J9.9 (Pin_9)
- net ENABLE_M2: now also J12.4 (Pin_4)
- net Echo1: now also J12.6 (Pin_6)
- net Echo2: now also J10.1 (Pin_1)
- net Echo3: now also J10.4 (Pin_4)
- net GND: now also H2.1, J11.2 (Pin_2), J11.3 (Pin_3), J9.4 (Pin_4)
- net RX: now also J10.8 (Pin_8)
- net SERVO: now also J10.2 (Pin_2)
- net STEP_M1: now also J9.7 (Pin_7)
- net STEP_M2: now also J10.5 (Pin_5)
- net TX: now also J10.7 (Pin_7)
- net Trig1: now also J12.5 (Pin_5)
- net Trig2: now also J9.10 (Pin_10)
- net Trig3: now also J10.6 (Pin_6)
- no-connect marks 52 -> 25
Other:
- note added: "Microcontrôleur"
- note removed: "Microcontrôleur STM32"
- moved on the sheet: H2, J6, J7, M1

Commit message: Version finale du pcb
Other:
- note added: "Microcontrôleur STM32 Nucleo F401RE"
- note added: "Source de puissance & Alimentation"
- note removed: "Microcontrôleur"
- note removed: "Source de puissance"
- moved on the sheet: A1, A2, C7, C8, H1, H2, J1, J10, J11, J12, J2, J3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
