File: PCB/PCB_HaSBot/robot2.kicad_pcb (KiCad board)
At the start: 2 copper layers, 71.6 x 73 mm, 17 parts, among them J1 Conn_01x04, J2 Conn_01x04, J3 Conn_01x04, J4 Conn_01x04, J5 Conn_01x04, J6 Conn_01x04, J7 Conn_01x04, J8 Screw_Terminal_01x02, M1 Motor_Servo, U1 STM32F401RETx, U3 L7805

Commit message: Version 2.0 du PCB
Parts:
- removed U1: STM32F401RETx, Package_QFP:LQFP-64_10x10mm_P0.5mm
- added H3: MountingHole_Pad, MountingHole:MountingHole_3.2mm_M3_DIN965_Pad, F.Cu at (142.2, 78.5)
- added J10: Conn_01x08, Connector_PinHeader_2.54mm:PinHeader_1x08_P2.54mm_Vertical, F.Cu at (166.4, 114.5)
- added J11: Conn_01x08, Connector_PinHeader_2.54mm:PinHeader_1x08_P2.54mm_Vertical, F.Cu at (118.2, 114.4)
- added J12: Conn_01x06, Connector_PinHeader_2.54mm:PinHeader_1x06_P2.54mm_Vertical, F.Cu at (118.1, 132.2)
- added J9: Conn_01x10, Connector_PinHeader_2.54mm:PinHeader_1x10_P2.54mm_Vertical, F.Cu at (166.4, 87.6)
- moved H1 2.11 mm to (125.1, 134.0)
- moved H2 0.58 mm to (160.0, 133.9)
- turned J8 to 0 degrees
Routing:
- net +9V: track 87.4 -> 125.7 mm, vias 1 -> 0
- net Echo2: track 55.1 -> 57.4 mm
- net ENABLE_M1: track 48.8 -> 51.0 mm
- net +5V: track 204.3 -> 202.1 mm
- net RX: track 75.4 -> 73.9 mm
- net DIR_M2: track 6.90 -> 8.12 mm
- net Echo3: track 10.8 -> 11.5 mm
- net DIR_M1: track 30.2 -> 30.8 mm

Commit message: Version finale du pcb
Parts:
- moved A2 6.26 mm to (148.3, 126.5)
- moved C8 6.26 mm to (154.9, 99.0)
- moved J3 6.26 mm to (151.7, 131.2)
- moved J5 6.26 mm to (116.8, 115.7)
- moved J4 6.26 mm to (137.4, 131.1)
- moved C11 6.26 mm to (141.2, 99.3)
- moved H3 6.26 mm to (148.0, 76.2)
- moved J1 6.26 mm to (164.7, 72.2)
- moved J10 6.26 mm to (172.3, 112.2)
- moved J11 6.26 mm to (124.0, 112.2)
- moved J7 6.26 mm to (178.7, 115.0)
- moved J9 6.26 mm to (172.2, 85.3)
- moved M1 6.26 mm to (178.9, 95.0)
- moved U3 6.26 mm to (150.5, 99.0)
- moved A1 6.26 mm to (127.0, 126.5)
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Routing:
- net +9V: track 125.7 -> 126.5 mm

Commit message: Correction du PCB
Parts:
- moved J7 7.14 mm to (179.7, 107.9), turned to -90 degrees
Routing:
- net +5V: track 202.1 -> 212.7 mm
- net Trig3: track 19.2 -> 15.7 mm
- net Echo3: track 11.5 -> 12.5 mm
- net +9V: track 126.5 -> 125.9 mm
- net SERVO: track 22.6 -> 23.1 mm
